File: devboard/devboard.kicad_sch (KiCad schematic)
At the start: 24 parts, among them J1 USB_B_Micro, J2 AVR-ISP-6, J3 Conn_01x15_Pin, J4 Conn_01x15_Pin, SW1 Pushbutton, SW2 SW_SPDT, SW3 SW_SPDT, U1 ATmega328P-P, U2 MCP2221AxST, U3 MCP1825S, Y1 Crystal

Commit message: Minor changes + added BOM
Parts:
- C3, C4: value 4.7μF -> 4.7uF
- C5: value 1μF -> 1uF; Manufacturer (none) -> KEMET; Mfr Part # (none) -> C0805C105K3RACTU
- D2: value LED_TX -> LED_YLW
- D3: value LED_RX -> LED_YLW
- D4: value LED -> LED_RED
- J1: value USB_B_Micro -> Micro-USB B
- R1: value 10KΩ -> 10K
- R2, R3, R4: value 200Ω -> 200R
- SW2, SW3: value SW_SPDT -> SPDT
- U2: value MCP2221AxST -> MCP2221A-I/ST; Manufacturer (none) -> Microchip; Mfr Part # (none) -> MCP2221A-I/ST
- Y1: value Crystal -> 16MHz Crystal
Other:
- moved on the sheet: C1, C2, D3, R1, R3
