File: rev_2/devboard/devboard.kicad_pcb (KiCad board)
At the start: 2 copper layers, 26.4 x 50.7 mm, 26 parts, among them J1 USB_C_Receptacle_USB2.0_16P, J2 AVR-ISP-6, J3 Conn_01x15_Pin, J4 Conn_01x15_Pin, SW1 Pushbutton, SW2 SPDT, SW3 SPDT, U1 ATmega328P-A, U2 MCP2221A-I/ST, U3 MCP1825S, Y1 Crystal_GND24

Commit message: Finished rev 2
Routing:
- net GND: track 5.00 -> 55.2 mm, vias 0 -> 2
- net /MISO: track 8.34 -> 37.7 mm
- net /SCK: track 10.0 -> 37.9 mm
- net /MOSI: track 9.06 -> 36.2 mm, vias 0 -> 1
- net /RST: track 15.3 -> 35.2 mm, vias 0 -> 1
- net /VDD_UART: track 55.2 -> 56.6 mm
Other:
- board text added: "ADC6"
- board text added: "ADC7"
- board text added: "AREF"
- board text added: "GND"
- board text added: "MISO"
- board text added: "MOSI"
- board text added: "PB0"
- board text added: "PB1"
- board text added: "PB2"
- board text added: "PC0"
- board text added: "PC1"
- board text added: "PC2"
- board text added: "PC3"
- board text added: "PC4"
- board text added: "PC5"
- board text added: "PD2"
- board text added: "PD3"
- board text added: "PD4"
- board text added: "PD5"
- board text added: "PD6"
- board text added: "PD7"
- board text added: "RESET"
- board text added: "RST"
- board text added: "RXD"
- board text added: "SCK"
- board text added: "TXD"
- board text added: "UART"
- board text added: "VCC"
- board text added: "VIN"
